Commit message: URDF fixed

File: generated/gazebo_launch/moveo/moveo.urdf (robot description, URDF)
Before this commit: robot moveo, 7 links, 7 joints
Links:
- added link world
Joints:
- joint j0: limit (none) -> lower=-3.14 upper=3.14 effort=100 velocity=1.0
- joint j1: limit (none) -> lower=-3.14 upper=3.14 effort=100 velocity=1.0
- joint j2: limit (none) -> lower=-3.14 upper=3.14 effort=100 velocity=1.0
- joint j3: limit (none) -> lower=-3.14 upper=3.14 effort=100 velocity=1.0
- joint j4: limit (none) -> lower=-3.14 upper=3.14 effort=100 velocity=1.0
- joint jtool: limit (none) -> lower=-3.14 upper=3.14 effort=100 velocity=1.0
